File: Kicad/placa/placa/placa.kicad_sch (KiCad schematic)
At the start: 4 parts, among them J1 Power, J2 Digital/PWM, J3 Analog, J4 Digital/PWM

Commit message: placa
Parts:
- added D1, D2, D3, D4: 1N4007, Diode_THT:D_DO-41_SOD81_P10.16mm_Horizontal, symbol Diode:1N4007
- added Q1: BC237, Package_TO_SOT_THT:TO-92_Inline, symbol Transistor_BJT:BC237
- added R1, R2, R3: R, symbol Device:R
- added SW1, SW2: SW_SPST, Button_Switch_THT:SW_PUSH_6mm, symbol Switch:SW_SPST
- added U1: PC817, Package_DIP:DIP-4_W7.62mm, symbol Isolator:PC817
- added U2: MOC3021M, symbol Relay_SolidState:MOC3021M
Connections:
- net 7 is gone; now on net +5V: J4.1 (Pin_1)
- net +5V: now also R2.2
- net GND: now also Q1.3 (E), U1.3
- net *10 renamed D10
- net *11 renamed D11
- net *3 renamed D3
- net *5 renamed D5
- net *6 renamed D6
- net *9 renamed D9
- net 12 renamed D12
- net 13 renamed D13
- net 2 renamed D2
- net 4 renamed D4
- net 8 renamed D8
- net AREF renamed AVDD
- net RX/0 renamed RX/D0
- net SCL/A5 renamed A5
- net A5: no longer J2.1 (Pin_1)
- net SDA/A4 renamed A4
- net A4: no longer J2.2 (Pin_2)
- net TX/1 renamed TX/D1
- new net: D1.1 (K), D2.1 (K), R1.1
- new net: D3.2 (A), D4.2 (A), U1.2
- new net: R3.2, U2.1
- new net: R2.1, U1.4
- new net: Q1.1 (C), U2.2
- new net: R1.2, U1.1
- new net L: D1.2 (A), D3.1 (K)
- new net N: D2.2 (A), D4.1 (K)
- new net SCL/D15: J2.1 (Pin_1)
- new net SDA/D14: J2.2 (Pin_2)

Commit message: placa y notas de aplicación
Parts:
- removed D1: 1N4007, Diode_THT:D_DO-41_SOD81_P10.16mm_Horizontal, symbol Diode:1N4007
- removed Q1: BC237, Package_TO_SOT_THT:TO-92_Inline, symbol Transistor_BJT:BC237
- removed SW1, SW2: SW_SPST, Button_Switch_THT:SW_PUSH_6mm, symbol Switch:SW_SPST
- removed U1: PC817, Package_DIP:DIP-4_W7.62mm, symbol Isolator:PC817
- removed U2: MOC3021M, symbol Relay_SolidState:MOC3021M
- added C1, C2: 0.1uF, symbol Device:C
- added D5: 1N4007, Diode_THT:D_DO-41_SOD81_P10.16mm_Horizontal, symbol Diode:1N4007
- added J5, J6, J7: Screw_Terminal_01x02, symbol Connector:Screw_Terminal_01x02
- added Q1, Q4: BT136-600, Package_TO_SOT_THT:TO-220-3_Vertical, symbol Triac_Thyristor:BT136-600
- added Q2, Q3: 2N7000, Package_TO_SOT_THT:TO-92_Inline, symbol Transistor_FET:2N7000
- added R10: 50, symbol Device:R
- added R11, R4: 200, symbol Device:R
- added R12, R5, R6: 100, symbol Device:R
- added R13, R14: 56k, symbol Device:R
- added R15: 10k, symbol Device:R
- added R7: 5, symbol Device:R
- added R8: 1M, symbol Device:R
- added R9: R, symbol Device:R
- added U1: 4N25, Package_DIP:DIP-6_W7.62mm, symbol Isolator:4N25
- added U2, U3: MOC3023M, symbol Relay_SolidState:MOC3023M
- R2: value R -> 1M
- R3: value R -> 5
Connections:
- net L is gone; now on an unnamed net: D3.1 (K)
- net SCL/D15 is gone; now on net SCL/A5: J2.1 (Pin_1)
- net SDA/D14 is gone; now on net SDA/A4: J2.2 (Pin_2)
- net +5V: now also R1.1, R15.1, R9.1; no longer J4.1 (Pin_1), R2.2
- net GND: now also R2.2, Q2.1 (S), Q3.1 (S), R8.2, U1.4
- net N: now also J7.1 (Pin_1), R14.2; no longer D2.2 (A), D4.1 (K)
- net at D2.1 (K): now also D4.1 (K), U1.1; no longer R1.1
- net at D4.2 (A): now also R14.1; no longer D3.2 (A)
- net at R3.2: now also R2.1, Q3.2 (G)
- net at R1.2: now also U2.1
- net A4 renamed SDA/A4
- net A5 renamed SCL/A5
- net AVDD renamed AREF
- net D10 renamed *10
- net D11 renamed *11
- net D12 renamed 12
- net D13 renamed 13
- net D2 renamed 2
- net D3 renamed *3
- net D4 renamed 4
- net D5 renamed *5
- net D6 renamed *6
- net D8 renamed 8
- net D9 renamed *9
- net RX/D0 renamed RX/0
- net TX/D1 renamed TX/1
- new net: C1.1, R12.1
- new net: C1.2, J6.2 (Pin_2), Q4.1 (A1), R10.2
- new net: C2.2, J5.2 (Pin_2), Q1.1 (A1), R6.2
- new net: R9.2, U3.1
- new net: Q3.3 (D), U2.2
- new net: Q1.3 (G), R6.1, U2.4
- new net: R4.1, U2.6
- new net: C2.1, R5.1
- new net: Q2.2 (G), R7.2, R8.1
- new net: Q2.3 (D), U3.2
- new net: Q4.3 (G), R10.1, U3.4
- new net: R11.1, U3.6
- new net: D2.2 (A), D5.1 (K), R13.1
- new net: D3.2 (A), D5.2 (A), U1.2
- new net: R15.2, U1.5
- new net 7: J4.1 (Pin_1)
- new net LINE: J5.1 (Pin_1), J6.1 (Pin_1), J7.2 (Pin_2), Q1.2 (A2), Q4.2 (A2), R11.2, R12.2, R13.2, R4.2, R5.2
