File: Kicad/placa/placa.kicad_sch (KiCad schematic)
At the start: 0 parts

Commit message: moved files
arreglé tema de kicad
Parts:
- added C1, C2: 0.1uF, symbol Device:C
- added D2, D3, D4, D5: 1N4007, Diode_THT:D_DO-41_SOD81_P10.16mm_Horizontal, symbol Diode:1N4007
- added J1: Power, Connector_PinSocket_2.54mm:PinSocket_1x08_P2.54mm_Vertical, symbol Connector_Generic:Conn_01x08
- added J2: Digital/PWM, Connector_PinSocket_2.54mm:PinSocket_1x10_P2.54mm_Vertical, symbol Connector_Generic:Conn_01x10
- added J3: Analog, Connector_PinSocket_2.54mm:PinSocket_1x06_P2.54mm_Vertical, symbol Connector_Generic:Conn_01x06
- added J4: Digital/PWM, Connector_PinSocket_2.54mm:PinSocket_1x08_P2.54mm_Vertical, symbol Connector_Generic:Conn_01x08
- added J5, J6, J7: Screw_Terminal_01x02, symbol Connector:Screw_Terminal_01x02
- added Q1, Q4: BT136-600, Package_TO_SOT_THT:TO-220-3_Vertical, symbol Triac_Thyristor:BT136-600
- added Q2, Q3: 2N7000, Package_TO_SOT_THT:TO-92_Inline, symbol Transistor_FET:2N7000
- added R1, R9: R, symbol Device:R
- added R10: 50, symbol Device:R
- added R11, R4: 200, symbol Device:R
- added R12, R5, R6: 100, symbol Device:R
- added R13, R14: 56k, symbol Device:R
- added R15: 10k, symbol Device:R
- added R2, R8: 1M, symbol Device:R
- added R3, R7: 5, symbol Device:R
- added U1: 4N25, Package_DIP:DIP-6_W7.62mm, symbol Isolator:4N25
- added U2, U3: MOC3023M, symbol Relay_SolidState:MOC3023M
Connections:
- new net: C1.1, R12.1
- new net: C1.2, J6.2 (Pin_2), Q4.1 (A1), R10.2
- new net: C2.2, J5.2 (Pin_2), Q1.1 (A1), R6.2
- new net: R9.2, U3.1
- new net: R1.2, U2.1
- new net: Q3.3 (D), U2.2
- new net: Q1.3 (G), R6.1, U2.4
- new net: R4.1, U2.6
- new net: C2.1, R5.1
- new net: Q3.2 (G), R2.1, R3.2
- new net: D3.1 (K), D4.2 (A), R14.1
- new net: Q2.2 (G), R7.2, R8.1
- new net: Q2.3 (D), U3.2
- new net: Q4.3 (G), R10.1, U3.4
- new net: R11.1, U3.6
- new net: D2.2 (A), D5.1 (K), R13.1
- new net: D3.2 (A), D5.2 (A), U1.2
- new net: R15.2, U1.5
- new net: D2.1 (K), D4.1 (K), U1.1
- new net *10: J2.8 (Pin_8)
- new net *11: J2.7 (Pin_7)
- new net *3: J4.5 (Pin_5)
- new net *5: J4.3 (Pin_3)
- new net *6: J4.2 (Pin_2)
- new net *9: J2.9 (Pin_9)
- new net +3V3: J1.4 (Pin_4)
- new net +5V: J1.5 (Pin_5), R1.1, R15.1, R9.1
- new net 12: J2.6 (Pin_6)
- new net 13: J2.5 (Pin_5)
- new net 2: J4.6 (Pin_6)
- new net 4: J4.4 (Pin_4)
- new net 7: J4.1 (Pin_1)
- new net 8: J2.10 (Pin_10)
- new net A0: J3.1 (Pin_1)
- new net A1: J3.2 (Pin_2)
- new net A2: J3.3 (Pin_3)
- new net A3: J3.4 (Pin_4)
- new net AREF: J2.3 (Pin_3)
- new net GND: J1.6 (Pin_6), J1.7 (Pin_7), J2.4 (Pin_4), Q2.1 (S), Q3.1 (S), R2.2, R8.2, U1.4
- new net IOREF: J1.2 (Pin_2)
- new net LINE: J5.1 (Pin_1), J6.1 (Pin_1), J7.2 (Pin_2), Q1.2 (A2), Q4.2 (A2), R11.2, R12.2, R13.2, R4.2, R5.2
- new net N: J7.1 (Pin_1), R14.2
- new net RX/0: J4.8 (Pin_8)
- new net SCL/A5: J2.1 (Pin_1), J3.6 (Pin_6)
- new net SDA/A4: J2.2 (Pin_2), J3.5 (Pin_5)
- new net TX/1: J4.7 (Pin_7)
- new net VCC: J1.8 (Pin_8)
- new net ~{RESET}: J1.3 (Pin_3)
- no-connect marks 0 -> 1
Other:
- note added: "* Indicates a PWM-capable pin"
