File: Kicad/placa alta tension/placa alta tension.kicad_pcb (KiCad board)
At the start: 2 copper layers, 66 x 53.3 mm, 4 parts, among them J1 Power, J2 Digital/PWM, J3 Analog, J4 Digital/PWM

Commit message: placa 220
Parts:
- removed J2: Digital/PWM, Connector_PinSocket_2.54mm:PinSocket_1x10_P2.54mm_Vertical
- removed J3: Analog, Connector_PinSocket_2.54mm:PinSocket_1x06_P2.54mm_Vertical
- removed J4: Digital/PWM, Connector_PinSocket_2.54mm:PinSocket_1x08_P2.54mm_Vertical
- added C1: 0.1uF, Capacitor_THT:C_Rect_L18.0mm_W9.0mm_P15.00mm_FKS3_FKP3, F.Cu at (154.5, 61.8)
- added C2: 0.1uF, Capacitor_THT:C_Rect_L18.0mm_W9.0mm_P15.00mm_FKS3_FKP3, F.Cu at (194.8, 62.8)
- added D1: 1N4007, Diode_THT:D_DO-41_SOD81_P10.16mm_Horizontal, F.Cu at (243.2, 126.5)
- added D2: 1N4007, Diode_THT:D_DO-41_SOD81_P10.16mm_Horizontal, F.Cu at (243.2, 130.8)
- added D3: 1N4007, Diode_THT:D_DO-41_SOD81_P10.16mm_Horizontal, F.Cu at (243.2, 135.0)
- added D4: 1N4007, Diode_THT:D_DO-41_SOD81_P10.16mm_Horizontal, F.Cu at (243.2, 139.2)
- added J6: Screw_Terminal_01x02, TerminalBlock_Phoenix:TerminalBlock_Phoenix_MKDS-1,5-2-5.08_1x02_P5.08mm_Horizontal, F.Cu at (196.8, 50.5)
- added J7: Screw_Terminal_01x02, TerminalBlock_Phoenix:TerminalBlock_Phoenix_MKDS-1,5-2-5.08_1x02_P5.08mm_Horizontal, F.Cu at (256.7, 137.4)
- added J9: Conn_01x05_Pin, Connector_PinHeader_2.54mm:PinHeader_1x05_P2.54mm_Vertical, F.Cu at (134.4, 100.0)
- added Q1: BT136-600, Package_TO_SOT_THT:TO-220-3_Vertical, F.Cu at (140.7, 48.0)
- added Q2: 2N7000, Package_TO_SOT_THT:TO-92_Inline, F.Cu at (139.8, 82.5)
- added Q3: BT136-600, Package_TO_SOT_THT:TO-220-3_Vertical, F.Cu at (178.2, 49.0)
- added Q4: 2N7000, Package_TO_SOT_THT:TO-92_Inline, F.Cu at (161.6, 88.5)
- added R1: 180, Resistor_THT:R_Axial_DIN0207_L6.3mm_D2.5mm_P7.62mm_Horizontal, F.Cu at (134.5, 87.3)
- added R10: 5, Resistor_THT:R_Axial_DIN0207_L6.3mm_D2.5mm_P7.62mm_Horizontal, F.Cu at (193.2, 99.3)
- added R11: 100, Resistor_THT:R_Axial_DIN0207_L6.3mm_D2.5mm_P7.62mm_Horizontal, F.Cu at (187.3, 70.5)
- added R12: 1M, Resistor_THT:R_Axial_DIN0207_L6.3mm_D2.5mm_P7.62mm_Horizontal, F.Cu at (218.7, 134.5)
- added R17: 56k, Resistor_THT:R_Axial_DIN0614_L14.3mm_D5.7mm_P15.24mm_Horizontal, F.Cu at (179.2, 140.0)
- added R18: 10k, Resistor_THT:R_Axial_DIN0207_L6.3mm_D2.5mm_P7.62mm_Horizontal, F.Cu at (218.7, 138.6)
- added R19: 56k, Resistor_THT:R_Axial_DIN0614_L14.3mm_D5.7mm_P15.24mm_Horizontal, F.Cu at (176.9, 151.0)
- added R2: 200, Resistor_THT:R_Axial_DIN0207_L6.3mm_D2.5mm_P7.62mm_Horizontal, F.Cu at (159.2, 66.1)
- added R3: 2.4k, Resistor_THT:R_Axial_DIN0614_L14.3mm_D5.7mm_P15.24mm_Horizontal, F.Cu at (166.0, 63.9)
- added R4: 5, Resistor_THT:R_Axial_DIN0207_L6.3mm_D2.5mm_P7.62mm_Horizontal, F.Cu at (139.0, 94.3)
- added R5: 100, Resistor_THT:R_Axial_DIN0207_L6.3mm_D2.5mm_P7.62mm_Horizontal, F.Cu at (147.1, 70.0)
- added R6: 1M, Resistor_THT:R_Axial_DIN0207_L6.3mm_D2.5mm_P7.62mm_Horizontal, F.Cu at (141.7, 87.2)
- added R7: 180, Resistor_THT:R_Axial_DIN0207_L6.3mm_D2.5mm_P7.62mm_Horizontal, F.Cu at (182.0, 92.3)
- added R8: 200, Resistor_THT:R_Axial_DIN0207_L6.3mm_D2.5mm_P7.62mm_Horizontal, F.Cu at (199.2, 65.9)
- added R9: 2.4k, Resistor_THT:R_Axial_DIN0614_L14.3mm_D5.7mm_P15.24mm_Horizontal, F.Cu at (205.8, 62.7)
- added U1: MOC3023M, Package_DIP:DIP-6_W7.62mm_Socket_LongPads, F.Cu at (153.2, 79.6)
- added U2: MOC3023M, Package_DIP:DIP-6_W7.62mm_Socket_LongPads, F.Cu at (193.0, 79.3)
- added U3: 4N25, Package_DIP:DIP-6_W7.62mm, F.Cu at (195.2, 110.5)
- J1: value Power -> Screw_Terminal_01x02; footprint Connector_PinSocket_2.54mm:PinSocket_1x08_P2.54mm_Vertical -> TerminalBlock_Phoenix:TerminalBlock_Phoenix_MKDS-1,5-2-5.08_1x02_P5.08mm_Horizontal
- moved J1 69.2 mm to (146.5, 30.8), turned to 180 degrees
Connections:
- J1 pad 1: unconnected-(J1-Pin_1-Pad1) -> LINE2
- J1 pad 2: /IOREF -> Net-(J1-Pin_2)
Other:
- board size 66 x 53.3 mm -> 104.8 x 77.8 mm

Commit message: placa
Parts:
- removed J6, J7: Screw_Terminal_01x02, TerminalBlock_Phoenix:TerminalBlock_Phoenix_MKDS-1,5-2-5.08_1x02_P5.08mm_Horizontal
- removed J9: Conn_01x05_Pin, Connector_PinHeader_2.54mm:PinHeader_1x05_P2.54mm_Vertical
- removed R17, R19: 56k, Resistor_THT:R_Axial_DIN0614_L14.3mm_D5.7mm_P15.24mm_Horizontal
- removed R18: 10k, Resistor_THT:R_Axial_DIN0207_L6.3mm_D2.5mm_P7.62mm_Horizontal
- added G***: LOGO, graphics:hotdog, B.Cu at (144.2, 124.5)
- added J2: Screw_Terminal_01x02, TerminalBlock_Phoenix:TerminalBlock_Phoenix_MKDS-1,5-2-5.08_1x02_P5.08mm_Horizontal, F.Cu at (101.4, 57.2)
- added J3: Screw_Terminal_01x02, TerminalBlock_Phoenix:TerminalBlock_Phoenix_MKDS-1,5-2-5.08_1x02_P5.08mm_Horizontal, F.Cu at (148.0, 56.5)
- added J4: Screw_Terminal_01x02, TerminalBlock_Phoenix:TerminalBlock_Phoenix_MKDS-1,5-2-5.08_1x02_P5.08mm_Horizontal, F.Cu at (122.0, 57.2)
- added R13: 5, Resistor_THT:R_Axial_DIN0207_L6.3mm_D2.5mm_P7.62mm_Horizontal, F.Cu at (134.0, 119.8)
- added R14: 100, Resistor_THT:R_Axial_DIN0207_L6.3mm_D2.5mm_P7.62mm_Horizontal, F.Cu at (123.2, 91.7)
- added R15: 1M, Resistor_THT:R_Axial_DIN0207_L6.3mm_D2.5mm_P7.62mm_Horizontal, F.Cu at (130.8, 119.8)
- J1: value Screw_Terminal_01x02 -> Conn_01x05_Socket; footprint TerminalBlock_Phoenix:TerminalBlock_Phoenix_MKDS-1,5-2-5.08_1x02_P5.08mm_Horizontal -> Connector_PinHeader_2.54mm:PinHeader_1x05_P2.54mm_Horizontal
- R1, R7: value 180 -> 56k; footprint Resistor_THT:R_Axial_DIN0207_L6.3mm_D2.5mm_P7.62mm_Horizontal -> Resistor_THT:R_Axial_DIN0614_L14.3mm_D5.7mm_P15.24mm_Horizontal
- R10: value 5 -> 180
- R11: value 100 -> 200
- R12: value 1M -> 2.4k; footprint Resistor_THT:R_Axial_DIN0207_L6.3mm_D2.5mm_P7.62mm_Horizontal -> Resistor_THT:R_Axial_DIN0614_L14.3mm_D5.7mm_P15.24mm_Horizontal
- R2: value 200 -> 180
- R3: value 2.4k -> 200; footprint Resistor_THT:R_Axial_DIN0614_L14.3mm_D5.7mm_P15.24mm_Horizontal -> Resistor_THT:R_Axial_DIN0207_L6.3mm_D2.5mm_P7.62mm_Horizontal
- R4: value 5 -> 10k
- R5: value 100 -> 2.4k; footprint Resistor_THT:R_Axial_DIN0207_L6.3mm_D2.5mm_P7.62mm_Horizontal -> Resistor_THT:R_Axial_DIN0614_L14.3mm_D5.7mm_P15.24mm_Horizontal
- R6: value 1M -> 5
- R8: value 200 -> 100
- R9: value 2.4k -> 1M; footprint Resistor_THT:R_Axial_DIN0614_L14.3mm_D5.7mm_P15.24mm_Horizontal -> Resistor_THT:R_Axial_DIN0207_L6.3mm_D2.5mm_P7.62mm_Horizontal
- U2: value MOC3023M -> 4N25
- U3: value 4N25 -> MOC3023M; footprint Package_DIP:DIP-6_W7.62mm -> Package_DIP:DIP-6_W7.62mm_Socket_LongPads
- moved D3 112.8 mm to (143.0, 83.1), turned to -90 degrees
- moved R9 111.7 mm to (109.8, 119.8)
- moved D4 111.4 mm to (147.0, 83.1), turned to -90 degrees
- moved R12 111.2 mm to (122.0, 79.5), turned to 90 degrees
- moved D2 100.0 mm to (150.5, 93.2), turned to 90 degrees
- moved R8 99.9 mm to (102.7, 91.5), turned to 0 degrees
- moved J1 97.4 mm to (130.2, 126.8), turned to -90 degrees
- moved D1 97.2 mm to (150.7, 96.7), turned to 180 degrees
- moved R2 79.8 mm to (100.2, 119.8)
- moved R10 75.1 mm to (121.0, 119.8)
- moved U3 74.2 mm to (121.0, 109.2), turned to 90 degrees
- moved R3 72.9 mm to (99.0, 92.6)
- moved R11 71.3 mm to (119.5, 92.7), turned to 90 degrees
- moved C2 66.9 mm to (130.0, 79.5), turned to 90 degrees
- moved Q3 61.3 mm to (129.1, 85.7), turned to 180 degrees
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Connections:
- C1 pad 2: Net-(J1-Pin_2) -> Net-(J2-Pin_2)
- C2 pad 2: Net-(J6-Pin_2) -> Net-(J4-Pin_2)
- J1 pad 1: LINE2 -> GND
- J1 pad 2: Net-(J1-Pin_2) -> +5V
- Q1 pad 1: Net-(J1-Pin_2) -> Net-(J2-Pin_2)
- Q1 pad 2: LINE2 -> LIGHT_LINE
- Q3 pad 1: Net-(J6-Pin_2) -> Net-(J4-Pin_2)
- Q3 pad 2: LINE1 -> DIMMING_LINE
- R1 pad 1: +5V -> Net-(D1-A)
- R1 pad 2: Net-(R1-Pad2) -> DIMMING_LINE
- R10 pad 1: /DIMM1 -> +5V
- R10 pad 2: Net-(Q4-G) -> Net-(R10-Pad2)
- R11 pad 1: Net-(Q3-G) -> Net-(R11-Pad1)
- R11 pad 2: Net-(J6-Pin_2) -> DIMMING_LINE
- R12 pad 1: Net-(Q4-G) -> Net-(C2-Pad1)
- R12 pad 2: GND -> DIMMING_LINE
- R2 pad 1: Net-(R2-Pad1) -> +5V
- R2 pad 2: LINE2 -> Net-(R2-Pad2)
- R3 pad 1: Net-(C1-Pad1) -> Net-(R3-Pad1)
- R3 pad 2: LINE2 -> LIGHT_LINE
- R4 pad 1: /DIMM2 -> +5V
- R4 pad 2: Net-(Q2-G) -> /ZCD
- R5 pad 1: Net-(Q1-G) -> Net-(C1-Pad1)
- R5 pad 2: Net-(J1-Pin_2) -> LIGHT_LINE
- R6 pad 1: Net-(Q2-G) -> /LIGHT
- R6 pad 2: GND -> Net-(Q2-G)
- R7 pad 1: +5V -> Net-(D2-A)
- R7 pad 2: Net-(R7-Pad2) -> N
- R8 pad 1: Net-(R8-Pad1) -> Net-(Q1-G)
- R8 pad 2: LINE1 -> Net-(J2-Pin_2)
- R9 pad 1: Net-(C2-Pad1) -> Net-(Q2-G)
- R9 pad 2: LINE1 -> GND
- U1 pad 1: Net-(R1-Pad2) -> Net-(R2-Pad2)
- U1 pad 6: Net-(R2-Pad1) -> Net-(R3-Pad1)
- U2 pad 1: Net-(R7-Pad2) -> Net-(D1-K)
- U2 pad 2: Net-(Q4-D) -> Net-(D3-A)
- U2 pad 4: Net-(Q3-G) -> GND
- U2 pad 5: unconnected-(U2-NC-Pad5) -> /ZCD
- U2 pad 6: Net-(R8-Pad1) -> unconnected-(U2-Pad6)
- U3 pad 1: Net-(D1-K) -> Net-(R10-Pad2)
- U3 pad 2: Net-(D3-A) -> Net-(Q4-D)
- U3 pad 4: GND -> Net-(Q3-G)
- U3 pad 5: /ZCD -> unconnected-(U3-NC-Pad5)
- U3 pad 6: unconnected-(U3-Pad6) -> Net-(R11-Pad1)
Routing:
- net GND: track 0.00 -> 97.3 mm, vias 0 -> 6
- net DIMMING_LINE: track 0.00 -> 78.5 mm
- net +5V: track 0.00 -> 75.4 mm, vias 0 -> 4
- net Net-(J2-Pin_2): track 0.00 -> 53.8 mm
- net Net-(J4-Pin_2): track 0.00 -> 53.2 mm
- net LIGHT_LINE: track 0.00 -> 42.8 mm
- net /ZCD: track 0.00 -> 31.3 mm
- net Net-(D1-A): track 0.00 -> 21.7 mm
- net Net-(Q4-G): track 0.00 -> 20.2 mm
- net Net-(Q3-G): track 0.00 -> 20.1 mm
- net Net-(Q2-G): track 0.00 -> 19.8 mm
- net Net-(Q1-G): track 0.00 -> 19.7 mm
- net /FAN: track 0.00 -> 16.0 mm
- net Net-(D3-A): track 0.00 -> 13.1 mm
- net /LIGHT: track 0.00 -> 11.0 mm
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- added copper zone on B.Cu, net GND
Other:
- board size 104.8 x 77.8 mm -> 60 x 80 mm
- board text added: "FAN"
- board text added: "IEC 9-12-2025 AC light dimmer"
- board text added: "LIGHT"
- board text added: "ZCD"

Commit message: simuklaciones ltspice y ajustes antes de comprar comps
Parts:
- removed Q1, Q3: BT136-600, Package_TO_SOT_THT:TO-220-3_Vertical
- added D5: Generic_Triac_A1A2G, Package_TO_SOT_THT:TO-220-3_Vertical, F.Cu at (108.5, 85.8)
- added D6: Generic_Triac_A1A2G, Package_TO_SOT_THT:TO-220-3_Vertical, F.Cu at (129.0, 85.8)
- R1, R7: value 56k -> 18k
- R11, R3: value 200 -> 220
- R14, R8: value 100 -> 220
- R4: value 10k -> 1k

Commit message: consulta Fede
Routing:
- net +5V: track 75.4 -> 77.2 mm
Changed lines of the file:
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@@
 		(grid_origin 96 51)
 		(pcbplotparams
-			(layerselection 0x00000000_00000000_5555555f_ff55d5ff)
-			(plot_on_all_layers_selection 0x00000000_00000000_00000000_00000000)
+			(layerselection 0x00000000_00000000_55555555_55555554)
+			(plot_on_all_layers_selection 0x00000000_00000000_0000000a_aa000004)
 			(disableapertmacros no)
 			(usegerberextensions no)
@@
 			(pdf_back_fp_property_popups yes)
 			(pdf_metadata yes)
-			(pdf_single_document no)
+			(pdf_single_document yes)
 			(dxfpolygonmode yes)
 			(dxfimperialunits yes)
@@
 			(psnegative no)
 			(psa4output no)
-			(plot_black_and_white yes)
+			(plot_black_and_white no)
 			(sketchpadsonfab no)
 			(plotpadnumbers no)
@@
 			(crossoutdnponfab yes)
 			(subtractmaskfromsilk no)
-			(outputformat 1)
+			(outputformat 4)
 			(mirror no)
 			(drillshape 0)
@@
 			(at 2.54 2.2 0)
 			(layer "F.Fab")
+			(hide yes)
 			(effects
 				(font
@@
 		(tags "Resistor Axial_DIN0207 series Axial Horizontal pin pitch 7.62mm 0.25W = 1/4W length 6.3mm diameter 2.5mm")
 		(property "Reference" "R3"
-			(at 3.81 -2.37 90)
+			(at 3.87 -2.5 90)
 			(layer "F.SilkS")
 			(effects
@@
 			(at 2.54 5.72 0)
 			(layer "F.Fab")
+			(hide yes)
 			(effects
 				(font
@@
 			(at 2.54 5.72 0)
 			(layer "F.Fab")
+			(hide yes)
 			(effects
 				(font
@@
 			(at 2.54 2.2 0)
 			(layer "F.Fab")
+			(hide yes)
 			(effects
 				(font
@@
 			(at 2.54 5.72 0)
 			(layer "F.Fab")
+			(hide yes)
 			(effects
 				(font
@@
 		)
 	)
+	(dimension
+		(type orthogonal)
+		(layer "F.Cu")
+		(pts
+			(xy 115.75 66.75) (xy 117.25 66.5)
+		)
+		(height -18.75)
+		(orientation 0)
+		(format
+			(prefix "")
+			(suffix "")
+			(units 3)
+			(units_format 1)
+			(precision 4)
+		)
+		(style
+			(thickness 0.15)
+			(arrow_length 1.27)
+			(text_position_mode 0)
+			(arrow_direction outward)
+			(extension_height 0.58642)
+			(extension_offset 0.5)
+			(keep_text_aligned yes)
+		)
+		(gr_text "1,5000 mm"
+			(at 116.5 46.2 0)
+			(layer "F.Cu")
+			(effects
+				(font
+					(size 1.5 1.5)
+					(thickness 0.3)
+				)
+			)
+		)
+	)
+	(dimension
+		(type orthogonal)
+		(layer "F.Cu")
+		(pts
+			(xy 99.19 102.325) (xy 98.75 109.75)
+		)
+		(height -9.44)
+		(orientation 1)
+		(format
+			(prefix "")
+			(suffix "")
+			(units 3)
+			(units_format 1)
+			(precision 4)
+		)
+		(style
+			(thickness 0.15)
+			(arrow_length 1.27)
+			(text_position_mode 0)
+			(arrow_direction outward)
+			(extension_height 0.58642)
+			(extension_offset 0.5)
+			(keep_text_aligned yes)
+		)
+		(gr_text "7,4250 mm"
+			(at 87.95 106.0375 90)
+			(layer "F.Cu")
+			(effects
+				(font
+					(size 1.5 1.5)
+					(thickness 0.3)
+				)
+			)
+		)
+	)
+	(dimension
+		(type orthogonal)
+		(layer "F.Cu")
+		(pts
+			(xy 102.92 57.1725) (xy 105 57.5)
+		)
+		(height -12.4225)
+		(orientation 0)
+		(format
+			(prefix "")
+			(suffix "")
+			(units 3)
+			(units_format 1)
+			(precision 4)
+		)
+		(style
+			(thickness 0.15)
+			(arrow_length 1.27)
+			(text_position_mode 0)
+			(arrow_direction outward)
+			(extension_height 0.58642)
+			(extension_offset 0.5)
+			(keep_text_aligned yes)
+		)
+		(gr_text "2,0800 mm"
+			(at 103.96 42.95 0)
+			(layer "F.Cu")
+			(effects
+				(font
+					(size 1.5 1.5)
+					(thickness 0.3)
+				)
+			)
+		)
+	)
 	(segment
 		(start 101.5 79.5)
@@
 	)
 	(segment
-		(start 113 124.25)
-		(end 107.75 124.25)
-		(width 1.27)
-		(layer "B.Cu")
-		(net 9)
-	)
-	(segment
-		(start 107.75 124.25)
-		(end 103.31 119.81)
-		(width 1.27)
-		(layer "B.Cu")
-		(net 9)
-	)
-	(segment
 		(start 121 119.81)
 		(end 121 122)
@@
 	)
 	(segment
-		(start 113.375 124.625)
-		(end 113 124.25)
+		(start 100.25 122.75)
+		(end 100.25 119.81)
 		(width 1.27)
 		(layer "B.Cu")
@@
 	)
 	(segment
-		(start 103.31 119.81)
-		(end 100.25 119.81)
+		(start 113 124.25)
+		(end 101.75 124.25)
 		(width 1.27)
 		(layer "B.Cu")
@@
 		(width 1.27)
 		(layer "B.Cu")
+		(net 9)
+	)
+	(segment
+		(start 101.75 124.25)
+		(end 100.25 122.75)
+		(width 1.27)
+		(layer "B.Cu")
+		(net 9)
+	)
+	(segment
+		(start 113.375 124.625)
+		(end 113 124.25)
+		(width 1.27)
+		(layer "B.Cu")

Commit message: placa v2
Parts:
- removed Q4: 2N7000, Package_TO_SOT_THT:TO-92_Inline
- added F1: Fuse, Fuse:Fuseholder_Clip-5x20mm_Bel_FC-203-22_Lateral_P17.80x5.00mm_D1.17mm_Horizontal, F.Cu at (201.7, 80.7)
- added F2: Fuse, Fuse:Fuseholder_Clip-5x20mm_Bel_FC-203-22_Lateral_P17.80x5.00mm_D1.17mm_Horizontal, F.Cu at (171.4, 80.6)
- added F3: Fuse, Fuse:Fuseholder_Clip-5x20mm_Bel_FC-203-22_Lateral_P17.80x5.00mm_D1.17mm_Horizontal, F.Cu at (140.2, 80.7)
- added Q1: 2N7000, Package_TO_SOT_THT:TO-92_Wide, F.Cu at (159.2, 117.7)
- added R16: 1M, Resistor_THT:R_Axial_DIN0207_L6.3mm_D2.5mm_P7.62mm_Horizontal, F.Cu at (170.0, 121.8)
- added RV1: Varistor, Varistor:RV_Disc_D15.5mm_W4.2mm_P7.5mm, F.Cu at (186.1, 64.0)
- added RV2: Varistor, Varistor:RV_Disc_D15.5mm_W4.2mm_P7.5mm, F.Cu at (163.5, 82.0)
- added RV3: Varistor, Varistor:RV_Disc_D15.5mm_W4.2mm_P7.5mm, F.Cu at (132.2, 82.1)
- added U4: MOC3023M, Package_DIP:DIP-6_W7.62mm_Socket_LongPads, F.Cu at (125.9, 109.5)
- D4: value 1N4007 -> Generic_Triac_A1A2G; footprint Diode_THT:D_DO-41_SOD81_P10.16mm_Horizontal -> Package_TO_SOT_THT:TO-220-3_Vertical
- D5: value Generic_Triac_A1A2G -> 1N4007; footprint Package_TO_SOT_THT:TO-220-3_Vertical -> Diode_THT:D_DO-41_SOD81_P10.16mm_Horizontal
- J1: value Conn_01x05_Socket -> Screw_Terminal_01x02; footprint Connector_PinHeader_2.54mm:PinHeader_1x05_P2.54mm_Horizontal -> TerminalBlock_Phoenix:TerminalBlock_Phoenix_MKDS-1,5-2-5.08_1x02_P5.08mm_Horizontal
- J4: value Screw_Terminal_01x02 -> Conn_01x05_Socket; footprint TerminalBlock_Phoenix:TerminalBlock_Phoenix_MKDS-1,5-2-5.08_1x02_P5.08mm_Horizontal -> Connector_PinHeader_2.54mm:PinHeader_1x05_P2.54mm_Horizontal
- Q2: footprint Package_TO_SOT_THT:TO-92_Inline -> Package_TO_SOT_THT:TO-92_Wide
- R1: value 18k -> 10k
- R10: value 180 -> 1M
- R11: value 220 -> 180
- R12: value 2.4k -> 220; footprint Resistor_THT:R_Axial_DIN0614_L14.3mm_D5.7mm_P15.24mm_Horizontal -> Resistor_THT:R_Axial_DIN0207_L6.3mm_D2.5mm_P7.62mm_Horizontal
- R13: value 5 -> 2.4k; footprint Resistor_THT:R_Axial_DIN0207_L6.3mm_D2.5mm_P7.62mm_Horizontal -> Resistor_THT:R_Axial_DIN0614_L14.3mm_D5.7mm_P15.24mm_Horizontal
- R14: value 220 -> 5
- R15, R9: value 1M -> 220
- R6: value 5 -> 2k; footprint Resistor_THT:R_Axial_DIN0207_L6.3mm_D2.5mm_P7.62mm_Horizontal -> Resistor_THT:R_Axial_DIN0411_L9.9mm_D3.6mm_P12.70mm_Horizontal
- R7: value 18k -> 5; footprint Resistor_THT:R_Axial_DIN0614_L14.3mm_D5.7mm_P15.24mm_Horizontal -> Resistor_THT:R_Axial_DIN0207_L6.3mm_D2.5mm_P7.62mm_Horizontal
- R8: value 220 -> 10k; footprint Resistor_THT:R_Axial_DIN0207_L6.3mm_D2.5mm_P7.62mm_Horizontal -> Resistor_THT:R_Axial_DIN0614_L14.3mm_D5.7mm_P15.24mm_Horizontal
- U3: value MOC3023M -> 74HC14; footprint Package_DIP:DIP-6_W7.62mm_Socket_LongPads -> Package_DIP:DIP-14_W7.62mm_Socket_LongPads
- moved J4 100.5 mm to (204.4, 114.6)
- moved J2 93.6 mm to (195.0, 56.5), turned to 180 degrees
- moved D5 83.9 mm to (192.4, 82.5), turned to -90 degrees
- moved R8 82.4 mm to (182.4, 70.6)
- moved J1 76.8 mm to (161.3, 56.5), turned to 180 degrees
- moved U3 73.1 mm to (193.8, 115.6), turned to -90 degrees
- moved R6 70.6 mm to (179.8, 97.2), turned to 0 degrees
- moved R5 66.2 mm to (167.6, 75.4), turned to 180 degrees
- moved R9 59.6 mm to (165.1, 97.8), turned to 180 degrees
- moved C1 59.2 mm to (167.5, 67.4), turned to 180 degrees
- moved R14 57.8 mm to (170.2, 125.2), turned to 180 degrees
- moved U1 56.6 mm to (157.0, 109.5)
- moved R2 53.4 mm to (153.6, 117.0)
- moved R3 53.0 mm to (152.0, 94.2), turned to 0 degrees
- moved Q2 52.1 mm to (157.9, 122.8)
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Connections:
- C1 pad 2: Net-(D5-A1) -> /HV11
- D2 pad 2: Net-(D2-A) -> /HV9
- D4 pad 1: Net-(D2-A) -> /HV11
- D4 pad 2: Net-(D3-A) -> Net-(D4-A2)
- D5 pad 1: Net-(D5-A1) -> /HV9
- D5 pad 2: LIGHT_LINE -> Net-(D3-A)
- D6 pad 2: DIMMING_LINE -> Net-(D6-A2)
- J1 pad 1: GND -> LIGHT_LINE
- J1 pad 2: +5V -> /HV11
- J2 pad 1: LIGHT_LINE -> Net-(J2-Pin_1)
- J2 pad 2: Net-(D5-A1) -> Net-(J2-Pin_2)
- J3 pad 1: N -> DIMMING_LINE
- J3 pad 2: DIMMING_LINE -> Net-(D6-A1)
- J4 pad 1: DIMMING_LINE -> GND
- J4 pad 2: Net-(D6-A1) -> +5V
- R1 pad 2: DIMMING_LINE -> Net-(J2-Pin_2)
- R10 pad 1: +5V -> Net-(Q1-G)
- R10 pad 2: Net-(R10-Pad2) -> GND
- R11 pad 1: Net-(R11-Pad1) -> +5V
- R11 pad 2: DIMMING_LINE -> Net-(R11-Pad2)
- R12 pad 1: Net-(C2-Pad1) -> Net-(R12-Pad1)
- R12 pad 2: DIMMING_LINE -> Net-(D6-A2)
- R13 pad 1: /FAN -> Net-(C2-Pad1)
- R13 pad 2: Net-(Q4-G) -> Net-(D6-A2)
- R14 pad 1: Net-(D6-G) -> Net-(R14-Pad1)
- R14 pad 2: Net-(D6-A1) -> Net-(Q2-G)
- R15 pad 1: Net-(Q4-G) -> Net-(D6-G)
- R15 pad 2: GND -> Net-(D6-A1)
- R3 pad 2: LIGHT_LINE -> Net-(D4-A2)
- R4 pad 2: /ZCD -> Net-(R4-Pad2)
- R5 pad 2: LIGHT_LINE -> Net-(D4-A2)
- R6 pad 1: /LIGHT -> Net-(R6-Pad1)
- R6 pad 2: Net-(Q2-G) -> Net-(D3-A)
- R7 pad 1: Net-(D2-A) -> Net-(R7-Pad1)
- R7 pad 2: N -> Net-(Q1-G)
- R8 pad 1: Net-(D5-G) -> /HV9
- R8 pad 2: Net-(D5-A1) -> N
- R9 pad 1: Net-(Q2-G) -> Net-(D4-G)
- R9 pad 2: GND -> /HV11
- U1 pad 2: Net-(Q2-D) -> Net-(Q1-D)
- U1 pad 4: Net-(D5-G) -> Net-(D4-G)
- U2 pad 2: Net-(D3-A) -> Net-(R6-Pad1)
- U2 pad 5: /ZCD -> Net-(R4-Pad2)
- U3 pad 1: Net-(R10-Pad2) -> GND
- U3 pad 2: Net-(Q4-D) -> unconnected-(U3-Pad2)
- U3 pad 3: unconnected-(U3-NC-Pad3) -> GND
- U3 pad 4: Net-(D6-G) -> unconnected-(U3-Pad4)
- U3 pad 5: unconnected-(U3-NC-Pad5) -> GND
- U3 pad 6: Net-(R11-Pad1) -> unconnected-(U3-Pad6)
Routing:
- net /HV11: track 0.00 -> 61.2 mm
- net DIMMING_LINE: track 78.5 -> 21.6 mm
- net Net-(D5-A1): track 53.8 -> 0.00 mm
- net Net-(D4-A2): track 0.00 -> 50.3 mm
- net Net-(D6-A2): track 0.00 -> 49.9 mm
- net Net-(R4-Pad2): track 0.00 -> 33.9 mm
- net Net-(J2-Pin_2): track 0.00 -> 29.6 mm
- net Net-(Q2-D): track 5.84 -> 31.2 mm
- net Net-(D1-K): track 9.56 -> 34.9 mm
- net N: track 8.29 -> 30.9 mm
- net /HV9: track 0.00 -> 21.8 mm
- net Net-(R11-Pad2): track 0.00 -> 21.8 mm
- net LIGHT_LINE: track 42.8 -> 21.4 mm
- net Net-(Q4-G): track 20.2 -> 0.00 mm
- net Net-(D5-G): track 19.7 -> 0.00 mm
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- removed copper zone on B.Cu, net GND
Other:
- board size 60 x 80 mm -> 94 x 80 mm
- board text added: "IEC 12-2025 AC fan + light dimmer"
- board text removed: "IEC 9-12-2025 AC light dimmer"
