File: Kicad/placa dimmer/dimmer.kicad_sch (KiCad schematic)
At the start: 52 parts, among them J1 Screw_Terminal_01x02, J2 Screw_Terminal_01x02, J3 Screw_Terminal_01x02, J4 Conn_01x05_Socket, Q1 2N7000, Q2 2N7000, U1 MOC3023M, U2 4N25, U3 74HC14, U4 MOC3023M

Commit message: ajustes finales
verificación de simulación con LTSpice, cambio de planos.
Parts:
- R6: value 2k -> 2k2
- TP10, TP11, TP12, TP13, TP16, TP3, TP4, TP5, TP6, TP7, TP8, TP9: now fitted
Other:
- note added: "CD40106"
- note removed: "* Indicates a PWM-capable pin"
- title: (none) -> Dimmer PCB
Changed lines of the file:
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@@
 	(paper "A4")
 	(title_block
-		(date "mar. 31 mars 2015")
+		(title "Dimmer PCB")
+		(date "2025-12-28")
+		(rev "V0")
 	)
 	(rectangle
@@
 		)
 	)
-	(text "* Indicates a PWM-capable pin"
+	(text "CD40106"
 		(exclude_from_sim no)
-		(at 177.8 180.34 0)
+		(at 249.682 83.82 0)
 		(effects
 			(font
 				(size 1.27 1.27)
 			)
-			(justify left bottom)
 		)
 	)
@@
 	(wire
 		(pts
-			(xy 127 76.2) (xy 130.81 76.2)
+			(xy 124.46 73.66) (xy 130.81 73.66)
 		)
 		(stroke
@@
 	(wire
 		(pts
-			(xy 130.81 76.2) (xy 130.81 82.55)
+			(xy 130.81 73.66) (xy 130.81 82.55)
 		)
 		(stroke
@@
 	(global_label "DIMMING_LINE"
 		(shape input)
-		(at 127 76.2 180)
+		(at 124.46 73.66 180)
 		(fields_autoplaced yes)
 		(effects
@@
 		)
 		(property "Intersheetrefs" "${INTERSHEET_REFS}"
-			(at 110.8568 76.2 0)
+			(at 108.3168 73.66 0)
 			(effects
 				(font
@@
 		(in_bom yes)
 		(on_board yes)
-		(dnp yes)
+		(dnp no)
 		(property "Reference" "TP11"
 			(at 227.33 17.272 0)
@@
 		(in_bom yes)
 		(on_board yes)
-		(dnp yes)
+		(dnp no)
 		(property "Reference" "TP5"
 			(at 82.042 99.06 0)
@@
 		(in_bom yes)
 		(on_board yes)
-		(dnp yes)
+		(dnp no)
 		(property "Reference" "TP10"
 			(at 110.49 55.118 0)
@@
 			)
 		)
-		(property "Value" "2k"
-			(at 214.63 41.402 90)
+		(property "Value" "2k2"
+			(at 219.456 46.736 90)
 			(effects
 				(font
@@
 		(dnp no)
 		(property "Reference" "D5"
-			(at 214.63 41.148 0)
+			(at 217.678 41.148 0)
 			(effects
 				(font
@@
 		)
 		(property "Value" "1N4007"
-			(at 214.376 43.18 0)
+			(at 211.836 41.148 0)
 			(effects
 				(font
@@
 		(in_bom yes)
 		(on_board yes)
-		(dnp yes)
+		(dnp no)
 		(property "Reference" "TP13"
 			(at 250.19 32.512 0)
@@
 		(in_bom yes)
 		(on_board yes)
-		(dnp yes)
+		(dnp no)
 		(property "Reference" "TP3"
 			(at 105.41 76.962 0)
@@
 		(in_bom yes)
 		(on_board yes)
-		(dnp yes)
+		(dnp no)
 		(property "Reference" "TP6"
 			(at 87.63 76.962 0)
@@
 		(in_bom yes)
 		(on_board yes)
-		(dnp yes)
+		(dnp no)
 		(property "Reference" "TP8"
 			(at 82.042 45.72 0)
@@
 		(in_bom yes)
 		(on_board yes)
-		(dnp yes)
+		(dnp no)
 		(property "Reference" "TP4"
 			(at 107.95 108.458 0)
@@
 		(in_bom yes)
 		(on_board yes)
-		(dnp yes)
+		(dnp no)
 		(property "Reference" "TP12"
 			(at 229.87 50.038 0)
@@
 		(in_bom yes)
 		(on_board yes)
-		(dnp yes)
+		(dnp no)
 		(property "Reference" "TP7"
 			(at 87.63 23.622 0)
@@
 		(in_bom yes)
 		(on_board yes)
-		(dnp yes)
+		(dnp no)
 		(property "Reference" "TP9"
 			(at 107.95 23.622 0)
@@
 		(in_bom yes)
 		(on_board yes)
-		(dnp yes)
+		(dnp no)
 		(property "Reference" "TP16"
 			(at 254.508 40.64 0)
@@
 		(on_board yes)
 		(dnp no)
-		(fields_autoplaced yes)
 		(property "Reference" "F3"
-			(at 124.46 76.2 90)
+			(at 124.714 76.962 90)
 			(effects
 				(font
