File: Kicad/placa shield/placa shield.kicad_pcb (KiCad board)
At the start: 2 copper layers, 68.6 x 53.3 mm, 20 parts, among them J1 HC-05 connector, J2 Digital/PWM, J3 Power, J4 Analog, J5 Digital/PWM, J6 Conn_01x05_Pin, SW1 SW_Push, SW2 SW_Push, SW3 SW_Push, SW4 SW_Push, SW5 SW_DIP_x04

Commit message: start of shield
Parts:
- J6: value Conn_01x05_Pin -> Dimmer module
Other:
- board size 68.6 x 53.3 mm -> 100 x 100 mm
Changed lines of the file:
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@@
 			)
 		)
-		(property "Value" "Conn_01x05_Pin"
+		(property "Value" "Dimmer module"
 			(at 0 12.54 0)
 			(layer "F.Fab")
@@
 			(type solid)
 		)
-		(locked yes)
 		(layer "Edge.Cuts")
 	)
@@
 			(type solid)
 		)
-		(locked yes)
 		(layer "Edge.Cuts")
 	)
@@
 			(type solid)
 		)
-		(locked yes)
 		(layer "Edge.Cuts")
 	)
@@
 			(type solid)
 		)
-		(locked yes)
 		(layer "Edge.Cuts")
 	)
@@
 			(type solid)
 		)
-		(locked yes)
 		(layer "Edge.Cuts")
 	)
@@
 			(type solid)
 		)
-		(locked yes)
 		(layer "Edge.Cuts")
 	)
@@
 			(type solid)
 		)
-		(locked yes)
 		(layer "Edge.Cuts")
 	)
@@
 			(type solid)
 		)
-		(locked yes)
 		(layer "Edge.Cuts")
 	)
@@
 			(type solid)
 		)
-		(locked yes)
 		(layer "Edge.Cuts")
 	)
@@
 			(type solid)
 		)
-		(locked yes)
+		(layer "Edge.Cuts")
+	)
+	(gr_rect
+		(start 86 32)
+		(end 186 132)
+		(stroke
+			(width 0.15)
+			(type solid)
+		)
+		(fill no)
 		(layer "Edge.Cuts")
 	)
@@
 			(type solid)
 		)
-		(locked yes)
 		(layer "Edge.Cuts")
 	)
@@
 			(type solid)
 		)
-		(locked yes)
 		(layer "Edge.Cuts")
 	)
